Commit message: modify package path
Signed-off-by: Masaya Kataoka <ms.kataoka@gmail.com>

File: genesis_ros/urdf/h1/h1.urdf (robot description, URDF)
Before this commit: robot h1_description, 25 links, 24 joints
Links:
- link left_ankle_link: geometry collision box size=0.28 0.03 0.024; visual mesh filename=meshes/left_ankle_link.dae
- link left_elbow_link: geometry collision cylinder length=0.09 radius=0.03; visual mesh filename=meshes/left_elbow_link.dae
- link left_hip_pitch_link: geometry collision cylinder length=0.2 radius=0.05; visual mesh filename=meshes/left_hip_pitch_link.dae
- link left_hip_roll_link: geometry collision cylinder length=0.01 radius=0.02; visual mesh filename=meshes/left_hip_roll_link.dae
- link left_hip_yaw_link: geometry collision cylinder length=0.02 radius=0.01; visual mesh filename=meshes/left_hip_yaw_link.dae
- link left_knee_link: geometry collision cylinder length=0.2 radius=0.05; visual mesh filename=meshes/left_knee_link.dae
- link left_shoulder_pitch_link: geometry collision cylinder length=0.04 radius=0.03; visual mesh filename=meshes/left_shoulder_pitch_link.dae
- link left_shoulder_roll_link: geometry collision cylinder length=0.01 radius=0.04; visual mesh filename=meshes/left_shoulder_roll_link.dae
- link left_shoulder_yaw_link: geometry collision cylinder length=0.01 radius=0.04; visual mesh filename=meshes/left_shoulder_yaw_link.dae
- link logo_link: geometry visual mesh filename=meshes/logo_link.dae
- link pelvis: geometry collision sphere radius=0.05; visual mesh filename=meshes/pelvis.dae
- link right_ankle_link: geometry collision box size=0.28 0.03 0.024; visual mesh filename=meshes/right_ankle_link.dae
- link right_elbow_link: geometry collision cylinder length=0.09 radius=0.03; visual mesh filename=meshes/right_elbow_link.dae
- link right_hip_pitch_link: geometry collision cylinder length=0.2 radius=0.05; visual mesh filename=meshes/right_hip_pitch_link.dae
- link right_hip_roll_link: geometry collision cylinder length=0.01 radius=0.02; visual mesh filename=meshes/right_hip_roll_link.dae
- link right_hip_yaw_link: geometry collision cylinder length=0.02 radius=0.01; visual mesh filename=meshes/right_hip_yaw_link.dae
- link right_knee_link: geometry collision cylinder length=0.2 radius=0.05; visual mesh filename=meshes/right_knee_link.dae
- link right_shoulder_pitch_link: geometry collision cylinder length=0.04 radius=0.03; visual mesh filename=meshes/right_shoulder_pitch_link.dae
- link right_shoulder_roll_link: geometry collision cylinder length=0.01 radius=0.04; visual mesh filename=meshes/right_shoulder_roll_link.dae
- link right_shoulder_yaw_link: geometry collision cylinder length=0.01 radius=0.04; visual mesh filename=meshes/right_shoulder_yaw_link.dae
- link torso_link: geometry collision box size=0.08 0.16 0.1; visual mesh filename=meshes/torso_link.dae

File: genesis_ros/urdf/h1/h1_with_hand.urdf (robot description, URDF)
Before this commit: robot h1, 52 links, 51 joints
Links:
- link L_hand_base_link: geometry collision mesh filename=meshes/L_hand_base_link.STL; visual mesh filename=meshes/L_hand_base_link.dae
- link L_index_intermediate: geometry collision mesh filename=meshes/Link16_L.STL; visual mesh filename=meshes/Link16_L.dae
- link L_index_proximal: geometry collision mesh filename=meshes/Link15_L.STL; visual mesh filename=meshes/Link15_L.dae
- link L_middle_intermediate: geometry collision mesh filename=meshes/Link18_L.STL; visual mesh filename=meshes/Link18_L.dae
- link L_middle_proximal: geometry collision mesh filename=meshes/Link17_L.STL; visual mesh filename=meshes/Link17_L.dae
- link L_pinky_intermediate: geometry collision mesh filename=meshes/Link22_L.STL; visual mesh filename=meshes/Link22_L.dae
- link L_pinky_proximal: geometry collision mesh filename=meshes/Link21_L.STL; visual mesh filename=meshes/Link21_L.dae
- link L_ring_intermediate: geometry collision mesh filename=meshes/Link20_L.STL; visual mesh filename=meshes/Link20_L.dae
- link L_ring_proximal: geometry collision mesh filename=meshes/Link19_L.STL; visual mesh filename=meshes/Link19_L.dae
- link L_thumb_distal: geometry collision mesh filename=meshes/Link14_L.STL; visual mesh filename=meshes/Link14_L.dae
- link L_thumb_intermediate: geometry collision mesh filename=meshes/Link13_L.STL; visual mesh filename=meshes/Link13_L.dae
- link L_thumb_proximal: geometry collision mesh filename=meshes/Link12_L.STL; visual mesh filename=meshes/Link12_L.dae
- link L_thumb_proximal_base: geometry collision mesh filename=meshes/Link11_L.STL; visual mesh filename=meshes/Link11_L.dae
- link R_hand_base_link: geometry collision mesh filename=meshes/R_hand_base_link.STL; visual mesh filename=meshes/R_hand_base_link.dae
- link R_index_intermediate: geometry collision mesh filename=meshes/Link16_R.STL; visual mesh filename=meshes/Link16_R.dae
- link R_index_proximal: geometry collision mesh filename=meshes/Link15_R.STL; visual mesh filename=meshes/Link15_R.dae
- link R_middle_intermediate: geometry collision mesh filename=meshes/Link18_R.STL; visual mesh filename=meshes/Link18_R.dae
- link R_middle_proximal: geometry collision mesh filename=meshes/Link17_R.STL; visual mesh filename=meshes/Link17_R.dae
- link R_pinky_intermediate: geometry collision mesh filename=meshes/Link22_R.STL; visual mesh filename=meshes/Link22_R.dae
- link R_pinky_proximal: geometry collision mesh filename=meshes/Link21_R.STL; visual mesh filename=meshes/Link21_R.dae
- link R_ring_intermediate: geometry collision mesh filename=meshes/Link20_R.STL; visual mesh filename=meshes/Link20_R.dae
- link R_ring_proximal: geometry collision mesh filename=meshes/Link19_R.STL; visual mesh filename=meshes/Link19_R.dae
- link R_thumb_distal: geometry collision mesh filename=meshes/Link14_R.STL; visual mesh filename=meshes/Link14_R.dae
- link R_thumb_intermediate: geometry collision mesh filename=meshes/Link13_R.STL; visual mesh filename=meshes/Link13_R.dae
- link R_thumb_proximal: geometry collision mesh filename=meshes/Link12_R.STL; visual mesh filename=meshes/Link12_R.dae
- link R_thumb_proximal_base: geometry collision mesh filename=meshes/Link11_R.STL; visual mesh filename=meshes/Link11_R.dae
- link left_ankle_link: geometry collision box size=0.28 0.03 0.024; visual mesh filename=meshes/left_ankle_link.dae
- link left_elbow_link: geometry collision cylinder length=0.09 radius=0.03; visual mesh filename=meshes/left_elbow_link.dae
- link left_hand_link: geometry collision mesh filename=meshes/left_hand_link.STL; visual mesh filename=meshes/left_hand_link.dae
- link left_hip_pitch_link: geometry collision cylinder length=0.2 radius=0.05; visual mesh filename=meshes/left_hip_pitch_link.dae
- link left_hip_roll_link: geometry collision cylinder length=0.01 radius=0.02; visual mesh filename=meshes/left_hip_roll_link.dae
- link left_hip_yaw_link: geometry collision cylinder length=0.02 radius=0.01; visual mesh filename=meshes/left_hip_yaw_link.dae
- link left_knee_link: geometry collision cylinder length=0.2 radius=0.05; visual mesh filename=meshes/left_knee_link.dae
- link left_shoulder_pitch_link: geometry collision cylinder length=0.04 radius=0.03; visual mesh filename=meshes/left_shoulder_pitch_link.dae
- link left_shoulder_roll_link: geometry collision cylinder length=0.01 radius=0.04; visual mesh filename=meshes/left_shoulder_roll_link.dae
- link left_shoulder_yaw_link: geometry collision cylinder length=0.01 radius=0.04; visual mesh filename=meshes/left_shoulder_yaw_link.dae
- link logo_link: geometry visual mesh filename=meshes/logo_link.dae
- link pelvis: geometry collision sphere radius=0.05; visual mesh filename=meshes/pelvis.dae
- link right_ankle_link: geometry collision box size=0.28 0.03 0.024; visual mesh filename=meshes/right_ankle_link.dae
- link right_elbow_link: geometry collision cylinder length=0.09 radius=0.03; visual mesh filename=meshes/right_elbow_link.dae
- link right_hand_link: geometry collision mesh filename=meshes/right_hand_link.STL; visual mesh filename=meshes/right_hand_link.dae
- link right_hip_pitch_link: geometry collision cylinder length=0.2 radius=0.05; visual mesh filename=meshes/right_hip_pitch_link.dae
- link right_hip_roll_link: geometry collision cylinder length=0.01 radius=0.02; visual mesh filename=meshes/right_hip_roll_link.dae
- link right_hip_yaw_link: geometry collision cylinder length=0.02 radius=0.01; visual mesh filename=meshes/right_hip_yaw_link.dae
- link right_knee_link: geometry collision cylinder length=0.2 radius=0.05; visual mesh filename=meshes/right_knee_link.dae
- link right_shoulder_pitch_link: geometry collision cylinder length=0.04 radius=0.03; visual mesh filename=meshes/right_shoulder_pitch_link.dae
- link right_shoulder_roll_link: geometry collision cylinder length=0.01 radius=0.04; visual mesh filename=meshes/right_shoulder_roll_link.dae
- link right_shoulder_yaw_link: geometry collision cylinder length=0.01 radius=0.04; visual mesh filename=meshes/right_shoulder_yaw_link.dae
- link torso_link: geometry collision box size=0.08 0.16 0.1; visual mesh filename=meshes/torso_link.dae
